Commit message: feat(urdf): update RealSense D435 model to use color_optical_frame feat(urdf): enhance table model with improved material definitions  for RVIz

File: urdf/realsense_d435.urdf.xacro (robot description, xacro)
@@ -10,5 +10,5 @@
   <xacro:include filename="$(find sp3_panda_ctrl)/urdf/_materials.urdf.xacro" />
   <xacro:include filename="$(find sp3_panda_ctrl)/urdf/_usb_plug.urdf.xacro" />
-  <xacro:macro name="sensor_d435" params="parent *origin name:=camera use_nominal_extrinsics:=false add_plug:=false use_mesh:=true">
+  <xacro:macro name="sensor_d435" params="parent *origin name:=camera use_nominal_extrinsics:=true add_plug:=false use_mesh:=true">
     <xacro:property name="M_PI" value="3.1415926535897931" />
     <!-- The following values are approximate, and the camera node
@@ -65,7 +65,7 @@
       </visual>
       <collision>
-        <origin xyz="0 ${-d435_cam_depth_py} 0" rpy="0 0 0"/>
+        <origin xyz="-0.02 ${-d435_cam_depth_py} 0" rpy="0 0 0"/>
         <geometry>
-          <box size="${d435_cam_depth} ${d435_cam_width} ${d435_cam_height}"/>
+          <box size="0.055 ${d435_cam_width} ${d435_cam_height}"/>
         </geometry>
       </collision>
@@ -137,8 +137,7 @@
       </xacro:usb_plug>
     </xacro:if>
-  </xacro:macro>
     <!-- === GAZEBO CAMERA SENSOR === -->
-  <gazebo reference="camera_link">
-    <sensor name="camera_rgb_sensor" type="camera">
+  <gazebo reference="${name}_color_frame">
+    <sensor name="${name}_rgb_sensor" type="camera">
       <always_on>true</always_on>
       <update_rate>30.0</update_rate>
@@ -155,13 +154,14 @@
         </clip>
       </camera>
-      <plugin name="camera_controller" filename="libgazebo_ros_camera.so">
+      <plugin name="${name}_controller" filename="libgazebo_ros_camera.so">
         <always_on>true</always_on>
         <update_rate>30.0</update_rate>
-        <camera_name>camera</camera_name>
+        <camera_name>${name}</camera_name>
         <image_topic_name>image_raw</image_topic_name>
         <camera_info_topic_name>camera_info</camera_info_topic_name>
-        <frame_name>camera_link</frame_name>
+        <frame_name>${name}_color_frame</frame_name>
       </plugin>
     </sensor>
   </gazebo>
+  </xacro:macro>
 </robot>

File: urdf/table.urdf.xacro (robot description, xacro)
@@ -1,152 +1,154 @@
 <?xml version="1.0"?>
 <robot xmlns:xacro="http://www.ros.org/wiki/xacro" name="table">
-<xacro:macro name="table" params="parent:=world xyz:='0 0 0' rpy:='0 0 0'">
-  <!-- === TISCHKÖRPER (schwarz) === -->
-  <link name="table_base">
-    <visual>
-      <origin xyz="0 0 0.485" rpy="0 0 0"/>
-      <geometry>
-        <box size="1.395 1.315 0.57"/>
-      </geometry>
-      <material name="black"><color rgba="0 0 0 1"/></material>
-    </visual>
-    <collision>
-      <origin xyz="0 0 0.485" rpy="0 0 0"/>
-      <geometry>
-        <box size="1.395 1.315 0.57"/>
-      </geometry>
-    </collision>
-    <inertial>
-      <mass value="40.0"/>
-      <origin xyz="0 0 0.485" rpy="0 0 0"/>
-      <inertia ixx="1.0" ixy="0.0" ixz="0.0" iyy="1.0" iyz="0.0" izz="1.0"/>
-    </inertial>
-  </link>
-  <gazebo reference="table_base">
-    <material>Gazebo/Black</material>
-  </gazebo>
-  <!-- === TISCHPLATTE (grau) === -->
-  <link name="table_top">
-    <visual>
-      <origin xyz="0 0 0.77" rpy="0 0 0"/>
-      <geometry>
-        <box size="1.40 1.32 0.04"/>
-      </geometry>
-      <material name="black"><color rgba="1 1 1 1"/></material>
-    </visual>
-    <collision>
-      <origin xyz="0 0 0.77" rpy="0 0 0"/>
-      <geometry>
-        <box size="1.40 1.32 0.04"/>
-      </geometry>
-    </collision>
-    <inertial>
-      <mass value="10.0"/>
-      <origin xyz="0 0 0.77" rpy="0 0 0"/>
-      <inertia ixx="0.5" ixy="0.0" ixz="0.0" iyy="0.5" iyz="0.0" izz="0.5"/>
-    </inertial>
-  </link>
-  <gazebo reference="table_top">
-    <material>Gazebo/Grey</material>
-  </gazebo>
-  <!-- === TISCHBEINE (grau) === -->
-  <!-- Bein vorne links -->
-  <link name="table_leg_1">
-    <visual>
-      <origin xyz="-0.65 -0.61 0.395" rpy="0 0 0"/>
-      <geometry>
-        <box size="0.1 0.1 0.79"/>
-      </geometry>
-      <material name="black"><color rgba="0 0 0 1"/></material>
-    </visual>
-    <collision>
-      <origin xyz="-0.65 -0.61 0.395" rpy="0 0 0"/>
-      <geometry>
-        <box size="0.1 0.1 0.79"/>
-      </geometry>
-    </collision>
-    <inertial>
-      <mass value="1.0"/>
-      <origin xyz="-0.65 -0.61 0.395" rpy="0 0 0"/>
-      <inertia ixx="0.01" ixy="0.0" ixz="0.0" iyy="0.01" iyz="0.0" izz="0.01"/>
-    </inertial>
-  </link>
-  <gazebo reference="table_leg_1">
-    <material>Gazebo/Grey</material>
-  </gazebo>
-  <!-- Bein vorne rechts -->
-  <link name="table_leg_2">
-    <visual>
-      <origin xyz="0.65 -0.61 0.395" rpy="0 0 0"/>
-      <geometry>
-        <box size="0.1 0.1 0.79"/>
-      </geometry>
-      <material name="black"><color rgba="0 0 0 1"/></material>
-    </visual>
-    <collision>
-      <origin xyz="0.65 -0.61 0.395" rpy="0 0 0"/>
-      <geometry>
-        <box size="0.1 0.1 0.79"/>
-      </geometry>
-    </collision>
-    <inertial>
-      <mass value="1.0"/>
-      <origin xyz="0.65 -0.61 0.395" rpy="0 0 0"/>
-      <inertia ixx="0.01" ixy="0.0" ixz="0.0" iyy="0.01" iyz="0.0" izz="0.01"/>
-    </inertial>
-  </link>
-  <gazebo reference="table_leg_2">
-    <material>Gazebo/Grey</material>
-  </gazebo>
-  <!-- Bein hinten links -->
-  <link name="table_leg_3">
-    <visual>
-      <origin xyz="-0.65 0.61 0.395" rpy="0 0 0"/>
-      <geometry>
-        <box size="0.1 0.1 0.79"/>
-      </geometry>
-      <material name="black"><color rgba="0 0 0 1"/></material>
-    </visual>
-    <collision>
-      <origin xyz="-0.65 0.61 0.395" rpy="0 0 0"/>
-      <geometry>
-        <box size="0.1 0.1 0.79"/>
-      </geometry>
-    </collision>
-    <inertial>
-      <mass value="1.0"/>
-      <origin xyz="-0.65 0.61 0.395" rpy="0 0 0"/>
-      <inertia ixx="0.01" ixy="0.0" ixz="0.0" iyy="0.01" iyz="0.0" izz="0.01"/>
-    </inertial>
-  </link>
-  <gazebo reference="table_leg_3">
-    <material>Gazebo/Grey</material>
-  </gazebo>
-  <!-- Bein hinten rechts -->
-  <link name="table_leg_4">
-    <visual>
-      <origin xyz="0.65 0.61 0.395" rpy="0 0 0"/>
-      <geometry>
-        <box size="0.1 0.1 0.79"/>
-      </geometry>
-      <material name="black"><color rgba="0 0 0 1"/></material>
-    </visual>
-    <collision>
-      <origin xyz="0.65 0.61 0.395" rpy="0 0 0"/>
-      <geometry>
-        <box size="0.1 0.1 0.79"/>
-      </geometry>
-    </collision>
-    <inertial>
-      <mass value="1.0"/>
-      <origin xyz="0.65 0.61 0.395" rpy="0 0 0"/>
-      <inertia ixx="0.01" ixy="0.0" ixz="0.0" iyy="0.01" iyz="0.0" izz="0.01"/>
-    </inertial>
-  </link>
-  <gazebo reference="table_leg_4">
-    <material>Gazebo/Grey</material>
-  </gazebo>
-  <!-- === JOINTS === -->
-    <!-- Beine -->
+  <xacro:macro name="table" params="parent:=world xyz:='0 0 0' rpy:='0 0 0'">
+    <!-- === Farben für den Tisch in RVIZ === -->
+    <material name="mat_black">
+      <color rgba="0 0 0 1"/>
+    </material>
+    <material name="mat_grey">
+      <color rgba="0.6 0.6 0.6 1"/>
+    </material>
+    <!-- === TISCHKÖRPER (schwarz) === -->
+    <link name="table_base">
+      <visual>
+        <origin xyz="0 0 0.485" rpy="0 0 0"/>
+        <geometry>
+          <box size="1.395 1.315 0.57"/>
+        </geometry>
+        <material name="mat_black"/>
+      </visual>
+      <collision>
+        <origin xyz="0 0 0.485" rpy="0 0 0"/>
+        <geometry>
+          <box size="1.395 1.315 0.57"/>
+        </geometry>
+      </collision>
+      <inertial>
+        <mass value="40.0"/>
+        <origin xyz="0 0 0.485" rpy="0 0 0"/>
+        <inertia ixx="1.0" ixy="0.0" ixz="0.0" iyy="1.0" iyz="0.0" izz="1.0"/>
+      </inertial>
+    </link>
+    <gazebo reference="table_base">
+      <material>Gazebo/Black</material>
+    </gazebo>
+    <!-- === TISCHPLATTE (grau) === -->
+    <link name="table_top">
+      <visual>
+        <origin xyz="0 0 0.77" rpy="0 0 0"/>
+        <geometry>
+          <box size="1.40 1.32 0.04"/>
+        </geometry>
+        <material name="mat_grey"/>
+      </visual>
+      <collision>
+        <origin xyz="0 0 0.77" rpy="0 0 0"/>
+        <geometry>
+          <box size="1.40 1.32 0.04"/>
+        </geometry>
+      </collision>
+      <inertial>
+        <mass value="10.0"/>
+        <origin xyz="0 0 0.77" rpy="0 0 0"/>
+        <inertia ixx="0.5" ixy="0.0" ixz="0.0" iyy="0.5" iyz="0.0" izz="0.5"/>
+      </inertial>
+    </link>
+    <gazebo reference="table_top">
+      <material>Gazebo/Grey</material>
+    </gazebo>
+    <!-- === TISCHBEINE (grau) === -->
+    <link name="table_leg_1">
+      <visual>
+        <origin xyz="-0.65 -0.61 0.395" rpy="0 0 0"/>
+        <geometry>
+          <box size="0.1 0.1 0.79"/>
+        </geometry>
+        <material name="mat_grey"/>
+      </visual>
+      <collision>
+        <origin xyz="-0.65 -0.61 0.395" rpy="0 0 0"/>
+        <geometry>
+          <box size="0.1 0.1 0.79"/>
+        </geometry>
+      </collision>
+      <inertial>
+        <mass value="1.0"/>
+        <origin xyz="-0.65 -0.61 0.395" rpy="0 0 0"/>
+        <inertia ixx="0.01" ixy="0.0" ixz="0.0" iyy="0.01" iyz="0.0" izz="0.01"/>
+      </inertial>
+    </link>
+    <gazebo reference="table_leg_1">
+      <material>Gazebo/Grey</material>
+    </gazebo>
+    <link name="table_leg_2">
+      <visual>
+        <origin xyz="0.65 -0.61 0.395" rpy="0 0 0"/>
+        <geometry>
+          <box size="0.1 0.1 0.79"/>
+        </geometry>
+        <material name="mat_grey"/>
+      </visual>
+      <collision>
+        <origin xyz="0.65 -0.61 0.395" rpy="0 0 0"/>
+        <geometry>
+          <box size="0.1 0.1 0.79"/>
+        </geometry>
+      </collision>
+      <inertial>
+        <mass value="1.0"/>
+        <origin xyz="0.65 -0.61 0.395" rpy="0 0 0"/>
+        <inertia ixx="0.01" ixy="0.0" ixz="0.0" iyy="0.01" iyz="0.0" izz="0.01"/>
+      </inertial>
+    </link>
+    <gazebo reference="table_leg_2">
+      <material>Gazebo/Grey</material>
+    </gazebo>
+    <link name="table_leg_3">
+      <visual>
+        <origin xyz="-0.65 0.61 0.395" rpy="0 0 0"/>
+        <geometry>
+          <box size="0.1 0.1 0.79"/>
+        </geometry>
+        <material name="mat_grey"/>
+      </visual>
+      <collision>
+        <origin xyz="-0.65 0.61 0.395" rpy="0 0 0"/>
+        <geometry>
+          <box size="0.1 0.1 0.79"/>
+        </geometry>
+      </collision>
+      <inertial>
+        <mass value="1.0"/>
+        <origin xyz="-0.65 0.61 0.395" rpy="0 0 0"/>
+        <inertia ixx="0.01" ixy="0.0" ixz="0.0" iyy="0.01" iyz="0.0" izz="0.01"/>
+      </inertial>
+    </link>
+    <gazebo reference="table_leg_3">
+      <material>Gazebo/Grey</material>
+    </gazebo>
+    <link name="table_leg_4">
+      <visual>
+        <origin xyz="0.65 0.61 0.395" rpy="0 0 0"/>
+        <geometry>
+          <box size="0.1 0.1 0.79"/>
+        </geometry>
+        <material name="mat_grey"/>
+      </visual>
+      <collision>
+        <origin xyz="0.65 0.61 0.395" rpy="0 0 0"/>
+        <geometry>
+          <box size="0.1 0.1 0.79"/>
+        </geometry>
+      </collision>
+      <inertial>
+        <mass value="1.0"/>
+        <origin xyz="0.65 0.61 0.395" rpy="0 0 0"/>
+        <inertia ixx="0.01" ixy="0.0" ixz="0.0" iyy="0.01" iyz="0.0" izz="0.01"/>
+      </inertial>
+    </link>
+    <gazebo reference="table_leg_4">
+      <material>Gazebo/Grey</material>
+    </gazebo>
+    <!-- === JOINTS === -->
     <joint name="table_leg_1_joint" type="fixed">
       <parent link="table_base"/>
@@ -165,6 +167,4 @@
       <child link="table_leg_4"/>
     </joint>
-    <!-- Positionierung des Tisches relativ zur Welt oder Roboter -->
-    <!-- Verbindung des Tisches mit dem übergeordneten Link -->
     <joint name="table_base_to_top" type="fixed">
       <parent link="table_top"/>
