Commit message: feat(panda): add visual work surface to URDF model

File: urdf/panda.urdf.xacro (robot description, xacro)
@@ -60,3 +60,20 @@
     <child link="table_top"/>
     <origin xyz="0 0 -0.79" rpy="0 0 0"/>  </joint>
+  <!-- === VISUAL ONLY WORK SURFACE (NO COLLISION) === -->
+  <link name="work_surface_visual">
+    <visual>
+      <origin xyz="0.4 0.0 0.791" rpy="0 0 0"/>
+      <geometry>
+        <box size="0.22 0.30 0.002"/>
+      </geometry>
+      <material name="work_surface_blue">
+        <color rgba="0.1 0.4 0.9 0.35"/>
+      </material>
+    </visual>
+  </link>
+  <joint name="work_surface_visual_joint" type="fixed">
+    <parent link="table_top"/>
+    <child link="work_surface_visual"/>
+    <origin xyz="0 0 0" rpy="0 0 0"/>
+  </joint>
 </robot>

Commit message: feat(urdf): enhance panda URDF with dynamic table height and add dropoff markers

File: urdf/panda.urdf.xacro (robot description, xacro)
@@ -9,17 +9,20 @@
   <xacro:include filename="$(find sp3_panda_ctrl)/urdf/wall.urdf.xacro"/>
   <xacro:arg name="arm_id" default="panda" />
+  <!-- Parameters -->
+  <xacro:arg name="table_height" default="0.79"/>
+  <xacro:property name="table_height" value="$(arg table_height)"/>
   <!-- === FRANKA ROBOT === -->
   <xacro:franka_robot arm_id="$(arg arm_id)"
                       joint_limits="${xacro.load_yaml('$(find franka_description)/robots/panda/joint_limits.yaml')}"/>
-  <!-- === TABLE === -->
+  <!-- Environment -->
   <xacro:table parent="panda_link0"/>
-  <!-- === WALLS AROUND WORKSPACE === -->
   <xacro:spawn_walls parent="panda_link0"/>
-  <!-- === CAMERA MOUNT LINK === -->
+  <!-- Camera mount -->
   <link name="camera_mount">
     <visual>
       <origin xyz="0 0 0" rpy="0 0 0"/>
       <geometry>
-        <mesh filename="package://sp3_panda_ctrl/meshes/Panda_RealSenseD435_Camera_Mount.STL" scale="0.001 0.001 0.001"/>
+        <mesh filename="package://sp3_panda_ctrl/meshes/Panda_RealSenseD435_Camera_Mount.STL"
+              scale="0.001 0.001 0.001"/>
       </geometry>
       <material name="dark_grey">
@@ -30,6 +33,5 @@
       <origin xyz="0 0 0" rpy="0 0 0"/>
       <geometry>
-        <!-- Beispielhafte vereinfachte Box als Kollisionskörper -->
-        <box size="0.00 0.00 0.00"/>
+        <box size="0.0 0.0 0.0"/>
       </geometry>
     </collision>
@@ -40,5 +42,4 @@
     </inertial>
   </link>
-  <!-- === FIX CAMERA MOUNT TO PANDA HAND === -->
   <joint name="camera_mount_joint" type="fixed">
     <parent link="panda_hand"/>
@@ -46,33 +47,96 @@
     <origin xyz="0.063 0.03 -0.01" rpy="0 0 3.1461"/>
   </joint>
-  <!-- === MOUNT INTEL REALSENSE D435 CAMERA === -->
   <xacro:sensor_d435 parent="camera_mount">
     <origin xyz="0.025 0.03 0.05" rpy="0 -1.5708 0"/>
   </xacro:sensor_d435>
-  <!-- === SPAWN TRAFFIC LIGHT ON TABLE === -->
+  <!-- Objects on table -->
   <xacro:traffic_light parent="table_top" xyz="0.6 -0.72 0.77" rpy="0 0 0"/>
-  <!-- === SPAWN TWO LIDAR SENSORS ON TABLE === -->
   <xacro:lidar_sensor parent="table_top" xyz="-0.6 -0.72 0.77" rpy="0 0 0" prefix="lidar1_"/>
   <xacro:lidar_sensor parent="table_top" xyz="0.6 0.72 0.77" rpy="0 0 0" prefix="lidar2_"/>
-  <!-- === FIX TABLE TO BASE LINK (panda_link0) === -->
-  <joint name="world_to_table_top" type="fixed">
+  <!-- Table relative to panda base -->
+  <joint name="panda_base_to_table_top" type="fixed">
     <parent link="panda_link0"/>
     <child link="table_top"/>
-    <origin xyz="0 0 -0.79" rpy="0 0 0"/>  </joint>
-  <!-- === VISUAL ONLY WORK SURFACE (NO COLLISION) === -->
+    <origin xyz="0 0 -${table_height}" rpy="0 0 0"/>
+  </joint>
+  <!-- Convenience frame: z=0 lies on the table surface -->
+  <link name="table_surface"/>
+  <joint name="table_top_to_table_surface" type="fixed">
+    <parent link="table_top"/>
+    <child link="table_surface"/>
+    <origin xyz="0 0 ${table_height}" rpy="0 0 0"/>
+  </joint>
+  <!-- Visual-only work surface marker -->
   <link name="work_surface_visual">
     <visual>
-      <origin xyz="0.4 0.0 0.791" rpy="0 0 0"/>
+      <origin xyz="0 0 0" rpy="0 0 0"/>
       <geometry>
         <box size="0.22 0.30 0.002"/>
       </geometry>
-      <material name="work_surface_blue">
-        <color rgba="0.1 0.4 0.9 0.35"/>
+      <material name="work_surface_white">
+        <color rgba="1.0 1.0 1.0 0.5"/>
       </material>
     </visual>
+    <collision>
+      <origin xyz="0 0 0" rpy="0 0 0"/>
+      <geometry>
+        <box size="0.0 0.0 0.0"/>
+      </geometry>
+    </collision>
   </link>
-  <joint name="work_surface_visual_joint" type="fixed">
+  <joint name="table_top_to_work_surface_visual" type="fixed">
     <parent link="table_top"/>
     <child link="work_surface_visual"/>
+    <origin xyz="0.5 0 ${table_height}" rpy="0 0 0"/>
+  </joint>
+  <!-- Dropoff markers -->
+  <link name="dropoff_red_default">
+    <visual>
+      <origin xyz="0.2 -0.6 0.791" rpy="0 0 0"/>
+      <geometry>
+        <box size="0.07 0.07 0.002"/>
+      </geometry>
+      <material name="dropoff_red_default_mat">
+        <color rgba="1.0 0.0 0.0 1.0"/>
+      </material>
+    </visual>
+    <collision>
+      <origin xyz="0 0 0" rpy="0 0 0"/>
+      <geometry>
+        <box size="0.0 0.0 0.0"/>
+      </geometry>
+    </collision>
+  </link>
+  <gazebo reference="dropoff_red_default">
+    <material>Gazebo/Red</material>
+  </gazebo>
+  <joint name="table_top_to_dropoff_red_default" type="fixed">
+    <parent link="table_top"/>
+    <child link="dropoff_red_default"/>
+    <origin xyz="0 0 0" rpy="0 0 0"/>
+  </joint>
+  <link name="dropoff_blue_jackal">
+    <visual>
+      <origin xyz="-0.2 -0.6 0.791" rpy="0 0 0"/>
+      <geometry>
+        <box size="0.07 0.07 0.002"/>
+      </geometry>
+      <material name="dropoff_blue_jackal_mat">
+        <color rgba="0.0 0.0 1.0 1.0"/>
+      </material>
+    </visual>
+    <collision>
+      <origin xyz="0 0 0" rpy="0 0 0"/>
+      <geometry>
+        <box size="0.0 0.0 0.0"/>
+      </geometry>
+    </collision>
+  </link>
+  <gazebo reference="dropoff_blue_jackal">
+    <material>Gazebo/Blue</material>
+  </gazebo>
+  <joint name="table_top_to_dropoff_blue_jackal" type="fixed">
+    <parent link="table_top"/>
+    <child link="dropoff_blue_jackal"/>
     <origin xyz="0 0 0" rpy="0 0 0"/>
   </joint>

Commit message: fix(urdf): adjust dropoff marker positions for improved alignment

File: urdf/panda.urdf.xacro (robot description, xacro)
@@ -93,5 +93,5 @@
   <link name="dropoff_red_default">
     <visual>
-      <origin xyz="0.2 -0.6 0.791" rpy="0 0 0"/>
+      <origin xyz="0.0 -0.6 0.791" rpy="0 0 0"/>
       <geometry>
         <box size="0.07 0.07 0.002"/>
@@ -118,5 +118,5 @@
   <link name="dropoff_blue_jackal">
     <visual>
-      <origin xyz="-0.2 -0.6 0.791" rpy="0 0 0"/>
+      <origin xyz="-0.3 -0.6 0.791" rpy="0 0 0"/>
       <geometry>
         <box size="0.07 0.07 0.002"/>

Commit message: chore: update project references from sp3_panda_ctrl to sp4_panda_ctrl

File: urdf/panda.urdf.xacro (robot description, xacro)
@@ -3,9 +3,9 @@
   <!-- === INCLUDE NECESSARY XACRO FILES === -->
   <xacro:include filename="$(find franka_description)/robots/common/franka_robot.xacro"/>
-  <xacro:include filename="$(find sp3_panda_ctrl)/urdf/traffic_light.urdf.xacro"/>
-  <xacro:include filename="$(find sp3_panda_ctrl)/urdf/table.urdf.xacro"/>
-  <xacro:include filename="$(find sp3_panda_ctrl)/urdf/lidar_sensor.urdf.xacro"/>
-  <xacro:include filename="$(find sp3_panda_ctrl)/urdf/realsense_d435.urdf.xacro"/>
-  <xacro:include filename="$(find sp3_panda_ctrl)/urdf/wall.urdf.xacro"/>
+  <xacro:include filename="$(find sp4_panda_ctrl)/urdf/traffic_light.urdf.xacro"/>
+  <xacro:include filename="$(find sp4_panda_ctrl)/urdf/table.urdf.xacro"/>
+  <xacro:include filename="$(find sp4_panda_ctrl)/urdf/lidar_sensor.urdf.xacro"/>
+  <xacro:include filename="$(find sp4_panda_ctrl)/urdf/realsense_d435.urdf.xacro"/>
+  <xacro:include filename="$(find sp4_panda_ctrl)/urdf/wall.urdf.xacro"/>
   <xacro:arg name="arm_id" default="panda" />
   <!-- Parameters -->
@@ -23,5 +23,5 @@
       <origin xyz="0 0 0" rpy="0 0 0"/>
       <geometry>
-        <mesh filename="package://sp3_panda_ctrl/meshes/Panda_RealSenseD435_Camera_Mount.STL"
+        <mesh filename="package://sp4_panda_ctrl/meshes/Panda_RealSenseD435_Camera_Mount.STL"
               scale="0.001 0.001 0.001"/>
       </geometry>

File: urdf/realsense_d435.urdf.xacro (robot description, xacro)
@@ -8,6 +8,6 @@
 <robot name="sensor_d435" xmlns:xacro="http://ros.org/wiki/xacro">
   <!-- Includes -->
-  <xacro:include filename="$(find sp3_panda_ctrl)/urdf/_materials.urdf.xacro" />
-  <xacro:include filename="$(find sp3_panda_ctrl)/urdf/_usb_plug.urdf.xacro" />
+  <xacro:include filename="$(find sp4_panda_ctrl)/urdf/_materials.urdf.xacro" />
+  <xacro:include filename="$(find sp4_panda_ctrl)/urdf/_usb_plug.urdf.xacro" />
   <xacro:macro name="sensor_d435" params="parent *origin name:=camera use_nominal_extrinsics:=true add_plug:=false use_mesh:=true">
     <xacro:property name="M_PI" value="3.1415926535897931" />
@@ -53,5 +53,5 @@
           <origin xyz="${d435_zero_depth_to_glass + d435_glass_to_front} ${-d435_cam_depth_py} 0" rpy="${M_PI/2} 0 ${M_PI/2}"/>
           <geometry>
-            <mesh filename="package://sp3_panda_ctrl/meshes/d435.dae" />
+            <mesh filename="package://sp4_panda_ctrl/meshes/d435.dae" />
           </geometry>
         </xacro:if>

Commit message: feat(controller): update gripper heights and add close width command

File: urdf/panda.urdf.xacro (robot description, xacro)
@@ -45,5 +45,5 @@
     <parent link="panda_hand"/>
     <child link="camera_mount"/>
-    <origin xyz="0.063 0.03 -0.01" rpy="0 0 3.1461"/>
+    <origin xyz="0.065 0.03 0.0" rpy="0 0 3.1461"/>
   </joint>
   <xacro:sensor_d435 parent="camera_mount">
@@ -88,56 +88,5 @@
     <parent link="table_top"/>
     <child link="work_surface_visual"/>
-    <origin xyz="0.5 0 ${table_height}" rpy="0 0 0"/>
-  </joint>
-  <!-- Dropoff markers -->
-  <link name="dropoff_red_default">
-    <visual>
-      <origin xyz="0.0 -0.6 0.791" rpy="0 0 0"/>
-      <geometry>
-        <box size="0.07 0.07 0.002"/>
-      </geometry>
-      <material name="dropoff_red_default_mat">
-        <color rgba="1.0 0.0 0.0 1.0"/>
-      </material>
-    </visual>
-    <collision>
-      <origin xyz="0 0 0" rpy="0 0 0"/>
-      <geometry>
-        <box size="0.0 0.0 0.0"/>
-      </geometry>
-    </collision>
-  </link>
-  <gazebo reference="dropoff_red_default">
-    <material>Gazebo/Red</material>
-  </gazebo>
-  <joint name="table_top_to_dropoff_red_default" type="fixed">
-    <parent link="table_top"/>
-    <child link="dropoff_red_default"/>
-    <origin xyz="0 0 0" rpy="0 0 0"/>
-  </joint>
-  <link name="dropoff_blue_jackal">
-    <visual>
-      <origin xyz="-0.3 -0.6 0.791" rpy="0 0 0"/>
-      <geometry>
-        <box size="0.07 0.07 0.002"/>
-      </geometry>
-      <material name="dropoff_blue_jackal_mat">
-        <color rgba="0.0 0.0 1.0 1.0"/>
-      </material>
-    </visual>
-    <collision>
-      <origin xyz="0 0 0" rpy="0 0 0"/>
-      <geometry>
-        <box size="0.0 0.0 0.0"/>
-      </geometry>
-    </collision>
-  </link>
-  <gazebo reference="dropoff_blue_jackal">
-    <material>Gazebo/Blue</material>
-  </gazebo>
-  <joint name="table_top_to_dropoff_blue_jackal" type="fixed">
-    <parent link="table_top"/>
-    <child link="dropoff_blue_jackal"/>
-    <origin xyz="0 0 0" rpy="0 0 0"/>
+    <origin xyz="0.4 0 ${table_height}" rpy="0 0 0"/>
   </joint>
 </robot>

Commit message: wip(testing results): sweet can be picked by the panda,without using the width and yaw from the SP4-System

File: urdf/panda.urdf.xacro (robot description, xacro)
@@ -38,5 +38,5 @@
     <inertial>
       <origin xyz="0 0 0" rpy="0 0 0"/>
-      <mass value="0.3"/>
+      <mass value="0.0001"/>
       <inertia ixx="0.001" ixy="0.0" ixz="0.0" iyy="0.001" iyz="0.0" izz="0.001"/>
     </inertial>
@@ -88,5 +88,5 @@
     <parent link="table_top"/>
     <child link="work_surface_visual"/>
-    <origin xyz="0.4 0 ${table_height}" rpy="0 0 0"/>
+    <origin xyz="0.455 0.0325 ${table_height}" rpy="0 0 0"/>
   </joint>
 </robot>
